Commit message: first new branch

File: code/EGO-Planner-v2/swarm-playground/main_ws/src/planner/plan_manage/urdf/stereo_camera.urdf.xacro (robot description, xacro)
@@ -3,8 +3,8 @@
     <!-- camera -->
     <xacro:include filename="$(find ego_planner)/urdf/stereo_camera.gazebo.xacro"/>
-    <xacro:property name="stereo_z" value="0.05" />
-    <xacro:property name="stereo_y" value="0.07" />
-    <xacro:property name="stereo_x" value="0.05" />
-    <xacro:property name="object_height" value="1.25" />
+    <xacro:property name="stereo_z" value="0" />
+    <xacro:property name="stereo_y" value="0" />
+    <xacro:property name="stereo_x" value="0" />
+    <xacro:property name="object_height" value="3.5" />
     <!-- Used for fixing robot to Gazebo 'base_link' -->
     <link name="world"/>

Commit message: new comm

File: code/EGO-Planner-v2/swarm-playground/main_ws/src/planner/plan_manage/urdf/stereo_camera.urdf.xacro (robot description, xacro)
@@ -6,5 +6,5 @@
     <xacro:property name="stereo_y" value="0.07" />
     <xacro:property name="stereo_x" value="0.05" />
-    <xacro:property name="object_height" value="1.25" />
+    <xacro:property name="object_height" value="3.5" />
     <!-- Used for fixing robot to Gazebo 'base_link' -->
     <link name="world"/>
